File: usbB_4pin.brd (EAGLE design)
At the start: 100 x 80 mm, 13 parts, among them IC1 788TV, IC2 TINY13-20PU, X1 PN61729-S

Commit message: minor layout changes
Parts:
- removed JP1: (no value), pinhead:2X03
- moved R2 6.59 mm to (91.9, 10.7)
- moved R4 4.68 mm to (91.9, 16.3)
- moved LED1 2.97 mm to (77.2, 11.7)
- moved R3 2.79 mm to (91.7, 5.08)
- moved C3 2.54 mm to (69.8, 20.3)
Connections:
- removed net N$10: IC2.6, LED1.1
- removed net N$11: IC2.2, LED1.3
- new net N$3: IC2.2, LED1.1
- new net N$5: IC2.6, LED1.3
Routing:
- net N$3: track 0.00 -> 65.6 mm
- net N$11: track 64.8 -> 0.00 mm
- net N$9: track 54.7 -> 23.6 mm
- net N$5: track 0.00 -> 9.89 mm
- net N$10: track 8.94 -> 0.00 mm
- net GND: track 151.3 -> 159.9 mm
- net N$8: track 16.5 -> 12.0 mm
- net VCC: track 69.8 -> 67.3 mm
- net N$6: track 16.3 -> 17.0 mm
- net N$7: track 16.3 -> 15.7 mm
Changed lines of the file:
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@@
 <element name="C1" library="rcl" package="E2,5-6E" value="22µF" x="33.02" y="6.35" rot="R270"/>
 <element name="C2" library="rcl" package="C050-025X075" value="100nF" x="17.78" y="5.08" rot="R180"/>
-<element name="C3" library="rcl" package="C050-025X075" value="100nF" x="72.39" y="20.32"/>
+<element name="C3" library="rcl" package="C050-025X075" value="100nF" x="69.85" y="20.32"/>
 <element name="R1" library="resistor" package="0204/7" value="" x="50.8" y="12.7" rot="R180"/>
-<element name="R2" library="resistor" package="0204/7" value="150Ohm" x="88.9" y="16.51"/>
-<element name="R3" library="resistor" package="0204/7" value="91Ohm" x="88.9" y="5.08"/>
-<element name="R4" library="resistor" package="0204/7" value="91Ohm" x="88.9" y="12.7"/>
+<element name="R2" library="resistor" package="0204/7" value="150Ohm" x="91.948" y="10.668"/>
+<element name="R3" library="resistor" package="0204/7" value="91Ohm" x="91.694" y="5.08"/>
+<element name="R4" library="resistor" package="0204/7" value="91Ohm" x="91.948" y="16.256"/>
 <element name="IC1" library="linear" package="TO220V" value="788TV" x="22.86" y="12.7"/>
 <element name="IC2" library="atmel" package="DIL08" value="TINY13-20PU" x="62.23" y="8.89" rot="R270">
@@
 <attribute name="OC_FARNELL" value="9171550" x="36.83" y="-12.7" size="1.778" layer="27" rot="R270" display="off"/>
 </element>
-<element name="LED1" library="led" package="LRTB_G6SG" value="LRTB_G6SG" x="76.2" y="8.89" rot="SMR0"/>
+<element name="LED1" library="led" package="LRTB_G6SG" value="LRTB_G6SG" x="77.216" y="11.684" rot="SMR0"/>
 <element name="SV1" library="con-lstb" package="MA04-1" value="" x="44.45" y="5.08">
 <attribute name="OC_NEWARK" value="unknown" x="73.66" y="-29.21" size="1.778" layer="27" display="off"/>
@@
 <attribute name="OC_FARNELL" value="unknown" x="-6.35" y="-12.7" size="1.778" layer="27" rot="R270" display="off"/>
 </element>
-<element name="JP1" library="pinhead" package="2X03" value="" x="-9.144" y="4.064"/>
 </elements>
 <signals>
@@
 <wire x1="38.1" y1="2.54" x2="38.1" y2="1.27" width="0.4064" layer="16"/>
 <wire x1="38.1" y1="1.27" x2="43.18" y2="1.27" width="0.4064" layer="16"/>
-<wire x1="74.93" y1="20.32" x2="92.71" y2="20.32" width="0.4064" layer="16"/>
-<wire x1="92.71" y1="1.27" x2="58.42" y2="1.27" width="0.4064" layer="16"/>
+<wire x1="95.504" y1="1.27" x2="58.42" y2="1.27" width="0.4064" layer="16"/>
 <wire x1="58.42" y1="1.27" x2="58.42" y2="5.08" width="0.4064" layer="16"/>
 <wire x1="43.18" y1="5.08" x2="43.18" y2="1.27" width="0.4064" layer="16"/>
 <wire x1="43.18" y1="1.27" x2="58.42" y2="1.27" width="0.4064" layer="16"/>
-<wire x1="92.71" y1="20.32" x2="92.71" y2="16.51" width="0.4064" layer="16"/>
-<wire x1="92.71" y1="16.51" x2="92.71" y2="12.7" width="0.4064" layer="16"/>
-<wire x1="92.71" y1="12.7" x2="92.71" y2="5.08" width="0.4064" layer="16"/>
-<wire x1="92.71" y1="5.08" x2="92.71" y2="1.27" width="0.4064" layer="16"/>
+<wire x1="95.504" y1="5.08" x2="95.504" y2="1.27" width="0.4064" layer="16"/>
+<wire x1="72.39" y1="20.32" x2="95.758" y2="20.32" width="0.4064" layer="16"/>
+<wire x1="95.758" y1="20.32" x2="95.758" y2="16.256" width="0.4064" layer="16"/>
+<wire x1="95.758" y1="16.256" x2="95.758" y2="10.668" width="0.4064" layer="16"/>
+<wire x1="95.758" y1="10.668" x2="95.504" y2="10.668" width="0.4064" layer="16"/>
+<wire x1="95.504" y1="10.668" x2="95.504" y2="5.08" width="0.4064" layer="16"/>
 </signal>
 <signal name="VCC">
@@
 <wire x1="66.04" y1="16.51" x2="66.04" y2="12.7" width="0.4064" layer="16"/>
 <wire x1="66.04" y1="12.7" x2="66.04" y2="20.32" width="0.4064" layer="16"/>
-<wire x1="66.04" y1="20.32" x2="69.85" y2="20.32" width="0.4064" layer="16"/>
+<wire x1="66.04" y1="20.32" x2="67.31" y2="20.32" width="0.4064" layer="16"/>
 </signal>
 <signal name="N$4">
@@
 <contactref element="LED1" pad="5"/>
 <contactref element="R4" pad="1"/>
-<wire x1="82.55" y1="15.24" x2="76.2" y2="15.24" width="0.4064" layer="16"/>
-<wire x1="76.2" y1="15.24" x2="76.2" y2="10.415" width="0.4064" layer="16"/>
-<wire x1="82.55" y1="15.24" x2="82.55" y2="12.7" width="0.4064" layer="16"/>
-<wire x1="82.55" y1="12.7" x2="85.09" y2="12.7" width="0.4064" layer="16"/>
-<wire x1="76.2" y1="10.415" x2="76.2" y2="10.415" width="0" layer="19" extent="1-16"/>
+<wire x1="77.216" y1="13.209" x2="77.216" y2="17.78" width="0.4064" layer="16"/>
+<wire x1="77.216" y1="17.78" x2="88.138" y2="17.78" width="0.4064" layer="16"/>
+<wire x1="88.138" y1="17.78" x2="88.138" y2="16.256" width="0.4064" layer="16"/>
 </signal>
 <signal name="N$7">
 <contactref element="LED1" pad="2"/>
 <contactref element="R3" pad="1"/>
-<wire x1="76.2" y1="7.365" x2="76.2" y2="2.54" width="0.4064" layer="16"/>
-<wire x1="76.2" y1="2.54" x2="85.09" y2="2.54" width="0.4064" layer="16"/>
-<wire x1="85.09" y1="2.54" x2="85.09" y2="5.08" width="0.4064" layer="16"/>
-<wire x1="76.2" y1="7.365" x2="76.2" y2="7.365" width="0" layer="19" extent="1-16"/>
+<wire x1="87.884" y1="5.08" x2="77.216" y2="5.08" width="0.4064" layer="16"/>
+<wire x1="77.216" y1="5.08" x2="77.216" y2="10.159" width="0.4064" layer="16"/>
 </signal>
 <signal name="N$8">
 <contactref element="LED1" pad="6"/>
 <contactref element="R2" pad="1"/>
-<wire x1="85.09" y1="16.51" x2="73.55" y2="16.51" width="0.4064" layer="16"/>
-<wire x1="73.55" y1="16.51" x2="73.55" y2="11.59" width="0.4064" layer="16"/>
-<wire x1="78.85" y1="11.59" x2="73.55" y2="11.59" width="0" layer="19" extent="1-16"/>
-</signal>
-<signal name="N$9">
-<contactref element="IC2" pad="3"/>
-<contactref element="LED1" pad="4"/>
-<wire x1="58.42" y1="7.62" x2="63.5" y2="7.62" width="0.4064" layer="16"/>
-<wire x1="63.5" y1="7.62" x2="63.5" y2="8.89" width="0.4064" layer="16"/>
-<wire x1="63.5" y1="8.89" x2="69.85" y2="8.89" width="0.4064" layer="16"/>
-<wire x1="69.85" y1="8.89" x2="69.85" y2="17.78" width="0.4064" layer="16"/>
-<wire x1="69.85" y1="17.78" x2="87.63" y2="17.78" width="0.4064" layer="16"/>
-<wire x1="87.63" y1="17.78" x2="87.63" y2="11.43" width="0.4064" layer="16"/>
-<wire x1="87.63" y1="11.43" x2="78.85" y2="11.43" width="0.4064" layer="16"/>
-<wire x1="78.85" y1="11.43" x2="78.85" y2="11.59" width="0.4064" layer="16"/>
-<wire x1="73.55" y1="11.59" x2="78.85" y2="11.59" width="0" layer="19" extent="1-16"/>
-</signal>
-<signal name="N$10">
-<contactref element="IC2" pad="6"/>
-<contactref element="LED1" pad="1"/>
-<wire x1="66.04" y1="7.62" x2="73.55" y2="7.62" width="0.4064" layer="16"/>
-<wire x1="73.55" y1="7.62" x2="73.55" y2="6.19" width="0.4064" layer="16"/>
-<wire x1="78.85" y1="6.19" x2="73.55" y2="6.19" width="0" layer="19" extent="1-16"/>
-</signal>
-<signal name="N$11">
-<contactref element="IC2" pad="2"/>
-<contactref element="LED1" pad="3"/>
-<wire x1="58.42" y1="10.16" x2="60.96" y2="10.16" width="0.4064" layer="16"/>
-<wire x1="60.96" y1="10.16" x2="60.96" y2="11.43" width="0.4064" layer="16"/>
-<wire x1="60.96" y1="11.43" x2="68.58" y2="11.43" width="0.4064" layer="16"/>
-<wire x1="68.58" y1="11.43" x2="68.58" y2="19.05" width="0.4064" layer="16"/>
-<wire x1="68.58" y1="19.05" x2="90.17" y2="19.05" width="0.4064" layer="16"/>
-<wire x1="90.17" y1="19.05" x2="90.17" y2="7.62" width="0.4064" layer="16"/>
-<wire x1="90.17" y1="7.62" x2="78.85" y2="7.62" width="0.4064" layer="16"/>
-<wire x1="78.85" y1="7.62" x2="78.85" y2="6.19" width="0.4064" layer="16"/>
-<wire x1="73.55" y1="6.19" x2="78.85" y2="6.19" width="0" layer="19" extent="1-16"/>
+<wire x1="79.866" y1="14.384" x2="88.138" y2="14.384" width="0.4064" layer="16"/>
+<wire x1="88.138" y1="14.384" x2="88.138" y2="10.668" width="0.4064" layer="16"/>
 </signal>
 <signal name="N$12">
@@
 </polygon>
 </signal>
+<signal name="N$3">
+<contactref element="IC2" pad="2"/>
+<contactref element="LED1" pad="1"/>
+<wire x1="58.42" y1="10.16" x2="60.706" y2="10.16" width="0.4064" layer="16"/>
+<wire x1="60.706" y1="10.16" x2="60.706" y2="11.43" width="0.4064" layer="16"/>
+<wire x1="60.706" y1="11.43" x2="70.358" y2="11.43" width="0.4064" layer="16"/>
+<wire x1="70.358" y1="11.43" x2="70.358" y2="19.05" width="0.4064" layer="16"/>
+<wire x1="70.358" y1="19.05" x2="92.456" y2="19.05" width="0.4064" layer="16"/>
+<wire x1="92.456" y1="19.05" x2="92.456" y2="9.144" width="0.4064" layer="16"/>
+<wire x1="92.456" y1="9.144" x2="79.866" y2="9.144" width="0.4064" layer="16"/>
+<wire x1="79.866" y1="9.144" x2="79.866" y2="8.984" width="0.4064" layer="16"/>
+</signal>
+<signal name="N$5">
+<contactref element="IC2" pad="6"/>
+<contactref element="LED1" pad="3"/>
+<wire x1="66.04" y1="7.62" x2="74.566" y2="7.62" width="0.4064" layer="16"/>
+<wire x1="74.566" y1="7.62" x2="74.566" y2="8.984" width="0.4064" layer="16"/>
+</signal>
+<signal name="N$9">
+<contactref element="IC2" pad="3"/>
+<contactref element="LED1" pad="4"/>
+<wire x1="58.42" y1="7.62" x2="63.246" y2="7.62" width="0.4064" layer="16"/>
+<wire x1="63.246" y1="7.62" x2="63.246" y2="8.636" width="0.4064" layer="16"/>
+<wire x1="63.246" y1="8.636" x2="71.374" y2="8.636" width="0.4064" layer="16"/>
+<wire x1="71.374" y1="8.636" x2="71.374" y2="14.732" width="0.4064" layer="16"/>
+<wire x1="71.374" y1="14.732" x2="74.566" y2="14.732" width="0.4064" layer="16"/>
+<wire x1="74.566" y1="14.732" x2="74.566" y2="14.384" width="0.4064" layer="16"/>
+</signal>
 </signals>

Commit message: correct values
Parts:
- C1: value 22µF -> 33u
- C2: value 100nF -> 470n
- C3: value 100nF -> 100n
- R1: value (none) -> 10k
- R2: value 150Ohm -> 150
- R3, R4: value 91Ohm -> 91
Changed lines of the file:
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@@
 </autorouter>
 <elements>
-<element name="C1" library="rcl" package="E2,5-6E" value="22µF" x="33.02" y="6.35" rot="R270"/>
-<element name="C2" library="rcl" package="C050-025X075" value="100nF" x="17.78" y="5.08" rot="R180"/>
-<element name="C3" library="rcl" package="C050-025X075" value="100nF" x="69.85" y="20.32"/>
-<element name="R1" library="resistor" package="0204/7" value="" x="50.8" y="12.7" rot="R180"/>
-<element name="R2" library="resistor" package="0204/7" value="150Ohm" x="91.948" y="10.668"/>
-<element name="R3" library="resistor" package="0204/7" value="91Ohm" x="91.694" y="5.08"/>
-<element name="R4" library="resistor" package="0204/7" value="91Ohm" x="91.948" y="16.256"/>
+<element name="C1" library="rcl" package="E2,5-6E" value="33u" x="33.02" y="6.35" rot="R270"/>
+<element name="C2" library="rcl" package="C050-025X075" value="470n" x="17.78" y="5.08" rot="R180"/>
+<element name="C3" library="rcl" package="C050-025X075" value="100n" x="69.85" y="20.32"/>
+<element name="R1" library="resistor" package="0204/7" value="10k" x="50.8" y="12.7" rot="R180"/>
+<element name="R2" library="resistor" package="0204/7" value="150" x="91.948" y="10.668"/>
+<element name="R3" library="resistor" package="0204/7" value="91" x="91.694" y="5.08"/>
+<element name="R4" library="resistor" package="0204/7" value="91" x="91.948" y="16.256"/>
 <element name="IC1" library="linear" package="TO220V" value="788TV" x="22.86" y="12.7"/>
 <element name="IC2" library="atmel" package="DIL08" value="TINY13-20PU" x="62.23" y="8.89" rot="R270">
