File: usbB_isp_no_lm2940.brd (EAGLE design)
At the start: 100 x 80 mm, 9 parts, among them IC2 TINY13-20PU, X1 PN61729-S

Commit message: waste less space when printing
Parts:
- moved C3 4.47 mm to (44.1, 5.62)
- moved LED1 4.47 mm to (14.4, 9.00)
- moved R1 4.47 mm to (38.5, 13.5)
- moved IC2 4.47 mm to (37.0, 6.18)
- moved R2 4.47 mm to (26.0, 12.0)
- moved SV2 4.47 mm to (49.1, 9.01)
- moved X1 4.47 mm to (2.38, 8.91)
- moved R3 4.47 mm to (26.2, 5.81)
- moved R4 4.47 mm to (26.2, 14.6)
Other:
- board size 100 x 80 mm -> 56 x 20 mm
