File: usbB_isp_no_lm2940.sch (EAGLE design)
At the start: 9 parts, among them IC2 TINY13-20PU, X1 PN61729-S

Commit message: minor adjustments (tm)
Connections:
- net GND: now also X1.2
Changed lines of the file:
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@@
 <wire x1="0" y1="76.2" x2="0" y2="78.74" width="0.1524" layer="91"/>
 <junction x="0" y="76.2"/>
-<wire x1="0" y1="76.2" x2="0" y2="58.42" width="0.1524" layer="91"/>
+<wire x1="0" y1="76.2" x2="0" y2="66.04" width="0.1524" layer="91"/>
+<pinref part="X1" gate="G$1" pin="2"/>
+<wire x1="0" y1="66.04" x2="0" y2="58.42" width="0.1524" layer="91"/>
+<wire x1="-5.08" y1="66.04" x2="0" y2="66.04" width="0.1524" layer="91"/>
+<junction x="0" y="66.04"/>
 </segment>
 </net>

Commit message: wrong usb-pin *again and again and again and again …
Connections:
- net GND: now also X1.4; no longer X1.2
Changed lines of the file:
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@@
 <wire x1="0" y1="76.2" x2="0" y2="78.74" width="0.1524" layer="91"/>
 <junction x="0" y="76.2"/>
-<wire x1="0" y1="76.2" x2="0" y2="66.04" width="0.1524" layer="91"/>
-<pinref part="X1" gate="G$1" pin="2"/>
-<wire x1="0" y1="66.04" x2="0" y2="58.42" width="0.1524" layer="91"/>
-<wire x1="-5.08" y1="66.04" x2="0" y2="66.04" width="0.1524" layer="91"/>
-<junction x="0" y="66.04"/>
+<wire x1="0" y1="76.2" x2="0" y2="71.12" width="0.1524" layer="91"/>
+<pinref part="X1" gate="G$1" pin="4"/>
+<wire x1="0" y1="71.12" x2="0" y2="58.42" width="0.1524" layer="91"/>
+<wire x1="-5.08" y1="71.12" x2="0" y2="71.12" width="0.1524" layer="91"/>
+<junction x="0" y="71.12"/>
 </segment>
 </net>
